File: axoloti_sliders.brd (EAGLE design)
At the start: 111.7 x 66.5 mm, 27 parts

Commit message: wip
Parts:
- removed LED1, LED2, LED3, LED4: (no value), SparkFun-LED:LED3MM
- removed S4: SWITCH-MOMENTARY-2PTH, SparkFun-Electromechanical:TACTILE-PTH
- removed U$4: (no value), MusicThingModular:MOUNTING_HOLE
- added VR10, VR11, VR12: (no value), SparkFun-Electromechanical:SLIDER-SMALL
- S1, S2, S3, S5: value SWITCH-MOMENTARY-2PTH -> SWITCH-MOMENTARY-212MM; device SparkFun-Electromechanical:TACTILE-PTH -> SparkFun-Electromechanical:TACTILE-PTH-12MM
- moved S3 116.4 mm to (7.62, -62.2), turned to 0 degrees
- moved U$6 97.2 mm to (156.2, 61.0)
- moved S6 89.0 mm to (15.2, 26.7), turned to 270 degrees
- moved VR1 58.4 mm to (82.5, 19.1)
- moved VR3 58.4 mm to (102.9, 19.1)
- moved VR4 58.4 mm to (113.0, 19.1)
- moved VR5 58.4 mm to (123.2, 19.1)
- moved VR8 58.4 mm to (72.4, 19.1)
- moved VR2 58.4 mm to (92.7, 19.1)
- moved VR6 58.4 mm to (133.3, 19.1)
- moved VR7 58.4 mm to (143.5, 19.1)
- moved VR9 58.4 mm to (153.7, 19.1)
- moved U$1 57.1 mm to (109.2, 17.8)
- moved S5 55.0 mm to (15.2, 8.89)
- moved S1 54.2 mm to (29.2, 26.7), turned to 90 degrees
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Other:
- board size 111.7 x 66.5 mm -> 160 x 66.5 mm
