File: axoloti_sliders.sch (EAGLE design)
At the start: 22 parts

Commit message: wip
Parts:
- removed LED1, LED2, LED3, LED4: (no value), SparkFun-LED:LED3MM
- removed S4: SWITCH-MOMENTARY-2PTH, SparkFun-Electromechanical:SWITCH-MOMENTARY-2PTH
- added VR10, VR11, VR12: (no value), SparkFun-Electromechanical:SLIDER20MM
- S1, S2, S3, S5: value SWITCH-MOMENTARY-2PTH -> SWITCH-MOMENTARY-212MM; device SparkFun-Electromechanical:SWITCH-MOMENTARY-2PTH -> SparkFun-Electromechanical:SWITCH-MOMENTARY-212MM
Other:
- moved on the sheet: S1, S2, S3
Changed lines of the file:
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@@
 <part name="X4" library="SparkFun-Connectors" deviceset="M05" device="LOCK"/>
 <part name="X3" library="SparkFun-Connectors" deviceset="M07" device="LOCK"/>
-<part name="S1" library="SparkFun-Electromechanical" deviceset="SWITCH-MOMENTARY-2" device="PTH"/>
-<part name="S2" library="SparkFun-Electromechanical" deviceset="SWITCH-MOMENTARY-2" device="PTH"/>
-<part name="S3" library="SparkFun-Electromechanical" deviceset="SWITCH-MOMENTARY-2" device="PTH"/>
-<part name="S4" library="SparkFun-Electromechanical" deviceset="SWITCH-MOMENTARY-2" device="PTH"/>
-<part name="S5" library="SparkFun-Electromechanical" deviceset="SWITCH-MOMENTARY-2" device="PTH"/>
+<part name="S5" library="SparkFun-Electromechanical" deviceset="SWITCH-MOMENTARY-2" device="12MM" value="SWITCH-MOMENTARY-212MM"/>
 <part name="S6" library="SparkFun-Electromechanical" deviceset="SWITCH-MOMENTARY-2" device="12MM"/>
-<part name="LED1" library="SparkFun-LED" deviceset="LED" device="3MM"/>
-<part name="LED2" library="SparkFun-LED" deviceset="LED" device="3MM"/>
-<part name="LED3" library="SparkFun-LED" deviceset="LED" device="3MM"/>
-<part name="LED4" library="SparkFun-LED" deviceset="LED" device="3MM"/>
 <part name="VR8" library="SparkFun-Electromechanical" deviceset="SLIDER" device="20MM"/>
 <part name="VR1" library="SparkFun-Electromechanical" deviceset="SLIDER" device="20MM"/>
@@
 <part name="VR7" library="SparkFun-Electromechanical" deviceset="SLIDER" device="20MM"/>
 <part name="VR9" library="SparkFun-Electromechanical" deviceset="SLIDER" device="20MM"/>
+<part name="VR10" library="SparkFun-Electromechanical" deviceset="SLIDER" device="20MM"/>
+<part name="VR11" library="SparkFun-Electromechanical" deviceset="SLIDER" device="20MM"/>
+<part name="VR12" library="SparkFun-Electromechanical" deviceset="SLIDER" device="20MM"/>
+<part name="S1" library="SparkFun-Electromechanical" deviceset="SWITCH-MOMENTARY-2" device="12MM" value="SWITCH-MOMENTARY-212MM"/>
+<part name="S2" library="SparkFun-Electromechanical" deviceset="SWITCH-MOMENTARY-2" device="12MM" value="SWITCH-MOMENTARY-212MM"/>
+<part name="S3" library="SparkFun-Electromechanical" deviceset="SWITCH-MOMENTARY-2" device="12MM" value="SWITCH-MOMENTARY-212MM"/>
 </parts>
 <sheets>
@@
 <instance part="X4" gate="G$1" x="76.2" y="20.32"/>
 <instance part="X3" gate="G$1" x="101.6" y="17.78"/>
-<instance part="S1" gate="G$1" x="48.26" y="30.48"/>
-<instance part="S2" gate="G$1" x="48.26" y="20.32"/>
-<instance part="S3" gate="G$1" x="63.5" y="20.32"/>
-<instance part="S4" gate="G$1" x="63.5" y="30.48"/>
 <instance part="S5" gate="G$1" x="48.26" y="43.18"/>
 <instance part="S6" gate="G$1" x="111.76" y="91.44"/>
-<instance part="LED1" gate="G$1" x="127" y="78.74"/>
-<instance part="LED2" gate="G$1" x="124.46" y="66.04"/>
-<instance part="LED3" gate="G$1" x="124.46" y="53.34"/>
-<instance part="LED4" gate="G$1" x="124.46" y="30.48"/>
 <instance part="VR8" gate="G$1" x="160.02" y="35.56"/>
 <instance part="VR1" gate="G$1" x="154.94" y="60.96"/>
@@
 <instance part="VR7" gate="G$1" x="175.26" y="35.56"/>
 <instance part="VR9" gate="G$1" x="154.94" y="101.6"/>
+<instance part="VR10" gate="G$1" x="137.16" y="60.96"/>
+<instance part="VR11" gate="G$1" x="121.92" y="58.42"/>
+<instance part="VR12" gate="G$1" x="109.22" y="60.96"/>
+<instance part="S1" gate="G$1" x="48.26" y="50.8"/>
+<instance part="S2" gate="G$1" x="48.26" y="58.42"/>
+<instance part="S3" gate="G$1" x="48.26" y="66.04"/>
 </instances>
 <busses>
