File: axocore_top_from_mech.brd (EAGLE design)
At the start: 160 x 50 mm, 17 parts, among them U1 JOYSTICKPTH, X1 X1, X3 M02PTH, X4 M02PTH

Commit message: finalised layout, starting routing
Parts:
- removed S1, S2, S3: SWITCH-MOMENTARY-212MM, SparkFun-Electromechanical:TACTILE-PTH-12MM
- removed VR3, VR4, VR5: (no value), MusicThingModular:9MM_SNAP-IN_POT
- added BIG_S1, BIG_S2, BIG_S3: SWITCH-MOMENTARY-212MM, SparkFun-Electromechanical:TACTILE-PTH-12MM
- added LED1, LED2, LED3, LED4: (no value), SparkFun-LED:LED3MM
- added POT_PA2, POT_PA3, POT_PA4, VR7: (no value), MusicThingModular:9MM_SNAP-IN_POT
- added R1, R2, R3, R4: (no value), MusicThingModular:7MM_RESISTOR
- added SMALL_S1, SMALL_S2, SMALL_S3: SWITCH-MOMENTARY-2PTH, SparkFun-Electromechanical:TACTILE-PTH
- moved U1 1.27 mm to (20.3, 15.2), turned to 270 degrees
- renumbered VR1 to POT_PA7, VR2 to POT_PA6, VR6 to POT_PA5
Connections:
- new net CM: X1.31
- new net G: X1.32, X1.33
- new net GND: POT_PA2.1, POT_PA3.1, POT_PA4.1, POT_PA5.1, POT_PA6.1, POT_PA7.1, U1.H3, U1.V3, VR7.1, X1.14, X1.20, X1.28, X1.40, X1.6
- new net LIN+: X1.34
- new net LIN-: X1.35
- new net N$1: BIG_S3.1, SMALL_S3.1
- new net N$10: LED4.K, R4.1
- new net N$2: BIG_S3.3, SMALL_S3.3
- new net N$3: BIG_S2.1, SMALL_S2.1
- new net N$4: BIG_S2.3, SMALL_S2.3
- new net N$5: BIG_S1.1, SMALL_S1.1
- new net N$6: BIG_S1.3, SMALL_S1.3
- new net N$7: LED1.K, R1.2
- new net N$8: LED2.K, R2.2
- new net N$9: LED3.K, R3.2
- new net PA0: U1.H2, X1.16
- new net PA1: U1.V2, VR7.2, X1.17
- new net PA2: POT_PA2.2, X1.18
- new net PA3: POT_PA3.2, X1.19
- new net PA4: POT_PA4.2, X1.22
- new net PA5: POT_PA5.2, X1.23
- new net PA6: POT_PA6.2, X1.24
- new net PA7: POT_PA7.2, X1.25
- new net PB0: X1.26
- new net PB1: X1.27
- new net PB6: X1.2
- new net PB7: X1.3
- new net PB8: X1.4
- new net PB9: X1.5
- new net PC0: X1.8
- new net PC1: X1.9
- new net PC2: X1.10
- new net PC3: X1.11
- new net PC4: X1.12
- new net PC5: X1.13
- new net RIN+: X1.36
- new net RIN-: X1.37
- new net VDD: X1.1, X1.7
- new net VDDA: POT_PA2.3, POT_PA3.3, POT_PA4.3, POT_PA5.3, POT_PA6.3, POT_PA7.3, U1.H1, U1.V1, VR7.3, X1.15, X1.21
- new net VDDC: X1.29, X1.30
Routing:
- added copper zone on layer 16, net GND
Other:
- board text added: "PA0>>"
- board text added: "PA1>>"
- board text removed: "Axoloti Core board outline connector/pad locations"

Commit message: Completed routing
Parts:
- R1, R2, R3, R4: value (none) -> 1k
- turned LED_PWM_PB1 to 0 degrees
- turned LED_PWM_PB8 to 0 degrees
- turned LED_PWM_PB9 to 0 degrees
- renumbered LED1 to LED_PWM_PB1, LED2 to LED_PWM_PB8, LED3 to LED_PWM_PB9, LED4 to LED_PB0_PWM, SMALL_S1 to SW_PC1, SMALL_S2 to SW_PC2, SMALL_S3 to SW_PC3, U1 to _, VR7 to POT_PA1
Connections:
- removed net G: X1.32, X1.33
- removed net N$1: BIG_S3.1, SW_PC3.1
- removed net N$2: BIG_S3.3, SW_PC3.3
- removed net N$3: BIG_S2.1, SW_PC2.1
- removed net N$4: BIG_S2.3, SW_PC2.3
- removed net N$5: BIG_S1.1, SW_PC1.1
- removed net N$6: BIG_S1.3, SW_PC1.3
- removed net VDDC: X1.29, X1.30
- net GND: now also LED_PB0_PWM.K, LED_PWM_PB1.K, LED_PWM_PB8.K, LED_PWM_PB9.K
- net N$10: now also LED_PB0_PWM.A, R4.2; no longer LED_PB0_PWM.K, R4.1
- net N$7: now also LED_PWM_PB1.A; no longer LED_PWM_PB1.K
- net N$8: now also LED_PWM_PB8.A; no longer LED_PWM_PB8.K
- net N$9: now also LED_PWM_PB9.A; no longer LED_PWM_PB9.K
- net PB0: now also R4.1
- net PB1: now also R1.1
- net PB8: now also R2.1
- net PB9: now also R3.1
- net PC0: now also _.B2A
- net PC1: now also BIG_S1.3, SW_PC1.3
- net PC2: now also BIG_S2.3, SW_PC2.3
- net PC3: now also BIG_S3.3, SW_PC3.3
- net VDD: now also BIG_S1.1, BIG_S2.1, BIG_S3.1, SW_PC1.1, SW_PC2.1, SW_PC3.1, _.B1A; no longer X1.1
- net VDDA: no longer X1.21
Routing:
- net VDDA: track 0.00 -> 218.0 mm, vias 0 -> 3
- net VDD: track 0.00 -> 147.6 mm, vias 0 -> 1
- net PA1: track 0.00 -> 94.3 mm
- net PA0: track 0.00 -> 92.8 mm, vias 0 -> 1
- net PC3: track 0.00 -> 81.2 mm, vias 0 -> 1
- net PA5: track 0.00 -> 80.4 mm, vias 0 -> 1
- net PC2: track 0.00 -> 71.3 mm, vias 0 -> 1
- net PC1: track 0.00 -> 62.4 mm, vias 0 -> 1
- net PC0: track 0.00 -> 61.5 mm, vias 0 -> 1
- net N$10: track 0.00 -> 58.0 mm
- net PA6: track 0.00 -> 54.2 mm, vias 0 -> 1
- net PB8: track 0.00 -> 53.0 mm, vias 0 -> 1
- net PB1: track 0.00 -> 52.1 mm, vias 0 -> 1
- net PB9: track 0.00 -> 52.0 mm, vias 0 -> 1
- net N$9: track 0.00 -> 49.8 mm
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Other:
- board text removed: "IN"
- board text removed: "v1.1 only!"

Commit message: Rev 1 Complete and sent to OSHPark
Routing:
- net VDD: track 147.6 -> 146.1 mm
- net PC0: track 61.5 -> 60.0 mm
- net PC1: track 62.4 -> 61.8 mm
- net VDDA: track 218.0 -> 218.3 mm, vias 3 -> 1
Other:
- board text added: "AXOLOTI CONTROL 1"
- board text added: "Axoloti Control 1 Designed in Herne Hill, London by Tom Whitwell December 2015 CC-BY-SA musicthing.co.uk PCB Rev 1"
- board text added: "Inspiration & thanks: Johannes Taelman, Curtis Roads, Max Mathews, Laurie Spiegel, Jean Claude Risset, Lejaren Hillier, John Chowning, Laurie Anderson, Joel Chadabe, Miller Puckette, Paul Stoffregen, Ezra Buchla, Brian Crabtree, Kelli Cain, Suzanne Ciani, Tom Erbe, Carl Stone, Rob Hordijk, Hans Nordelius, Magnus Kjellander, Bjorn Leander, Christopher Richardson, Bengt Lilja."
- board text added: "Parts: PS3 thumb joystick 6 x 10k Linear D Shaft Pots Bourns PTV09A- 4020F-B103 Alps RK09K11310KB 3 x 12mm square tactile switches B3F-4050 = switch B32-1310 = black keycap B32-1320 = orange B32-1330 = yellow B32-1360 = white B32-1380 = red 4 x 1k Resistors 4 x 3mm LEDs 4 x 11mm M3 Hex Standoffs 2 x 2 pin Female Header 571-215297-2 40 pin Female Header"
